File: IO.sch (KiCad schematic (older format))
At the start: 0 parts

Commit message: Fix empty IO.sch file
Parts:
- added C10, C5, C6: 1µF, Capacitor_SMD:C_0805_2012Metric, symbol Device:C
- added C12, C13, C14, C3, C4, C7, C8, C9: 100nF, Capacitor_SMD:C_0603_1608Metric, symbol Device:C
- added D3: RX_R, Diode_SMD:D_0603_1608Metric, symbol Device:LED
- added D4: TX_G, Diode_SMD:D_0603_1608Metric, symbol Device:LED
- added J10: Bob-GY271, Connector_PinSocket_2.54mm:PinSocket_1x05_P2.54mm_Vertical, symbol Bobs-emt:Bob-GY271
- added J11: extPower, Connector_PinHeader_2.54mm:PinHeader_2x02_P2.54mm_Vertical, symbol Connector_Generic:Conn_02x02_Odd_Even
- added J12: I2C1, Connector_PinHeader_2.54mm:PinHeader_1x03_P2.54mm_Vertical, symbol Connector_Generic:Conn_01x03
- added J13: UART2, Connector_PinHeader_2.54mm:PinHeader_1x03_P2.54mm_Vertical, symbol Connector_Generic:Conn_01x03
- added J15: OW1, Connector_PinHeader_2.54mm:PinHeader_1x02_P2.54mm_Vertical, symbol Connector_Generic:Conn_01x02
- added J2: PI_SPI1, Pmod_Interface-emt:Pmod_Interface_Female6, symbol Pmod-Interface-emt:Pmod-Interface-SPI6
- added J3: Pmod-Interface-GPIO12, Pmod_Interface-emt:Pmod_Interface_Female12, symbol Pmod-Interface-emt:Pmod-Interface-GPIO12
- added J4: PI_GPIO12, Connector_PinHeader_2.54mm:PinHeader_2x06_P2.54mm_Vertical, symbol Connector_Generic:Conn_02x06_Odd_Even
- added J5: SPI1, Connector_PinHeader_2.54mm:PinHeader_1x06_P2.54mm_Vertical, symbol Connector_Generic:Conn_01x06
- added J6: Pmod-Interface-UART6, Pmod_Interface-emt:Pmod_Interface_Female6, symbol Pmod-Interface-emt:Pmod-Interface-UART6
- added J7: Pmod-I2C1, Pmod_Interface-emt:Pmod_Interface_Female6, symbol Pmod-Interface-emt:Pmod-Interface-I2C6
- added J8: Bob_GY291_ADXL345, Connector_PinSocket_2.54mm:PinSocket_1x08_P2.54mm_Vertical, symbol Bobs-emt:Bob_GY291_ADXL345
- added J9: Bob-DS18B20, Bobs-emt:Bob_DS18B20_Host, symbol Bobs-emt:Bob-DS18B20
- added JP1: OW_PULLUP_EN, Jumper:SolderJumper-2_P1.3mm_Open_TrianglePad1.0x1.5mm, symbol Jumper:SolderJumper_2_Open
- added JP2: I2C1_PULLUP_SDA, Jumper:SolderJumper-2_P1.3mm_Open_TrianglePad1.0x1.5mm, symbol Jumper:SolderJumper_2_Open
- added JP3: I2C1_PULLUP_SCL, Jumper:SolderJumper-2_P1.3mm_Open_TrianglePad1.0x1.5mm, symbol Jumper:SolderJumper_2_Open
- added JP4: OW1_3V3_EN, Jumper:SolderJumper-2_P1.3mm_Open_TrianglePad1.0x1.5mm, symbol Jumper:SolderJumper_2_Open
- added JP5: CS1Pulls, Jumper:SolderJumper-3_P2.0mm_Open_TrianglePad1.0x1.5mm, symbol Jumper:SolderJumper_3_Open
- added JP6: CS2Pulls, Jumper:SolderJumper-3_P2.0mm_Open_TrianglePad1.0x1.5mm, symbol Jumper:SolderJumper_3_Open
- added JP7: IO_SPI_CS_EN, Jumper:SolderJumper-3_P2.0mm_Open_TrianglePad1.0x1.5mm, symbol Jumper:SolderJumper_3_Open
- added R10, R11, R6, R7: 10k, Resistor_SMD:R_0603_1608Metric, symbol Device:R
- added R3: 4.7k, Resistor_SMD:R_0603_1608Metric, symbol Device:R
- added R4, R5: 2.2k, Resistor_SMD:R_0603_1608Metric, symbol Device:R
- added R8: 560, Resistor_SMD:R_0603_1608Metric, symbol Device:R
- added R9: 330, Resistor_SMD:R_0603_1608Metric, symbol Device:R
- added U2: DS18B20, Package_TO_SOT_THT:TO-92_Inline, symbol Sensor_Temperature:DS18B20
Connections:
- net labels added: +3V3, GND, io_i2c1_scl, io_i2c1_sda, io_io_adc_1, io_io_adc_2, io_io_io_1, io_io_io_2, io_io_io_3, io_io_io_4, io_io_io_5, io_io_io_6, io_ow1, io_spi1_miso, io_spi1_mosi, io_spi1_sclk, io_uart2_rx, io_uart2_tx, ~io_spi1_cs_1, ~io_spi1_cs_2
- wire segments 0 -> 160
- no-connect marks 0 -> 5
Other:
- note added: "External Power"
- note added: "I2C"
- note added: "IO1"
- note added: "Onewire1"
- note added: "SPI1"
- note added: "UART2"
