File: pmi-hw-bob2.kicad_pcb (KiCad board)
At the start: 2 copper layers, 54.6 x 87.6 mm, 57 parts, among them J1 Bob_St_N64_Morpho_Right, J10 Bob-GY271, J11 extPower, J12 I2C1, J13 UART2, J15 OW1, J2 PI_SPI1, J3 Pmod-Interface-GPIO12, J4 PI_GPIO12, J5 SPI1, J6 Pmod-Interface-UART6, J7 Pmod-I2C1, J8 Bob_GY291_ADXL345, J9 Bob-DS18B20, U1 MCP1703T-3302E_SOT23, U2 DS18B20

Commit message: Bump to version 1.2
Parts:
- JP4: value OW1_3V3_EN -> ParasiticPowerBridge; footprint Jumper:SolderJumper-2_P1.3mm_Open_TrianglePad1.0x1.5mm -> Jumper:SolderJumper-3_P2.0mm_Open_TrianglePad1.0x1.5mm_NumberLabels
- moved U2 3.51 mm to (105.4, 116.6)
- moved JP4 3.03 mm to (121.7, 118.0)
- moved C2 2.86 mm to (89.4, 90.4)
- moved D1 2.86 mm to (93.8, 88.9)
- moved D2 2.86 mm to (93.8, 90.8)
- moved R1 2.86 mm to (93.8, 86.9)
- moved R2 2.86 mm to (93.8, 92.7)
- moved C1 2.77 mm to (86.4, 86.7)
- moved U1 2.64 mm to (86.4, 90.5)
- moved JP1 2.06 mm to (100.4, 115.7)
- moved R3 2.06 mm to (103.1, 116.9)
Connections:
- J1 pad 1: Net-(J1-Pad1) -> (no net)
- J1 pad 10: Net-(J1-Pad10) -> (no net)
- J1 pad 16: Net-(J1-Pad16) -> (no net)
- J1 pad 17: Net-(J1-Pad17) -> (no net)
- J1 pad 18: Net-(J1-Pad18) -> (no net)
- J1 pad 19: Net-(J1-Pad19) -> (no net)
- J1 pad 21: Net-(J1-Pad21) -> (no net)
- J1 pad 23: Net-(J1-Pad23) -> (no net)
- J1 pad 25: Net-(J1-Pad25) -> (no net)
- J1 pad 27: Net-(J1-Pad27) -> (no net)
- J1 pad 29: Net-(J1-Pad29) -> (no net)
- J1 pad 31: Net-(J1-Pad31) -> (no net)
- J1 pad 33: Net-(J1-Pad33) -> (no net)
- J1 pad 36: Net-(J1-Pad36) -> (no net)
- J1 pad 38: Net-(J1-Pad38) -> (no net)
- J1 pad 7: Net-(J1-Pad7) -> (no net)
- J10 pad 5: Net-(J10-Pad5) -> (no net)
- J6 pad 1: Net-(J6-Pad1) -> (no net)
- J6 pad 4: Net-(J6-Pad4) -> (no net)
- J7 pad 1: Net-(J7-Pad1) -> (no net)
- J7 pad 2: Net-(J7-Pad2) -> (no net)
- J8 pad 4: Net-(J8-Pad4) -> (no net)
- J8 pad 5: Net-(J8-Pad5) -> (no net)
- JP4 pad 1: Net-(J9-Pad3) -> +3V3
- JP4 pad 2: +3V3 -> Net-(J9-Pad3)
Routing:
- net +3V3: track 296.9 -> 284.8 mm
- net /mcu_ow1: track 56.2 -> 53.1 mm
- net Net-(J9-Pad3): track 22.3 -> 24.9 mm
- net +5V: track 24.3 -> 23.1 mm
- net GND: vias 165 -> 162
Other:
- board text added: "PMI-BoB² V1.2 2021"
- board text added: "Parasitic Power"
- board text removed: "OW1 3V3 En"
- board text removed: "PMI-BoB² V1.1 2021"

Commit message: Bump to version 1.3
Parts:
- added H7: github.com-QR-Code, Symbol-emt:github-emtpb-pmi, B.Cu at (89.8, 89.7)
- U1: value MCP1703T-3302E_SOT23 -> MCP1703AT-3302E_SOT23
- moved H4 0.91 mm to (123.3, 133.3)
- renumbered C6 to C10, C7 to C11, C3 to C12, C8 to C13, C5 to C3, C10 to C4, C4 to C5, C13 to C6, C9 to C7, C14 to C8, C12 to C9, H6 to H5, H5 to H6, J2 to J10, J15 to J11, J6 to J12, J9 to J14, J4 to J2, J11 to J4, J12 to J6, J10 to J9, JP5 to JP1, JP6 to JP2, JP2 to JP3, JP3 to JP4, JP7 to JP5, JP1 to JP6, JP4 to JP7, R9 to R10, R3 to R11, R6 to R3, R7 to R4, R10 to R5, R11 to R6, R4 to R7, R5 to R8, R8 to R9
Connections:
- net /~mcu_spi1_cs1 renamed /~{mcu_spi1_cs1}
- net /~mcu_spi1_cs2 renamed /~{mcu_spi1_cs2}
- J1 pad 1: (no net) -> unconnected-(J1-Pad1)
- J1 pad 10: (no net) -> unconnected-(J1-Pad10)
- J1 pad 16: (no net) -> unconnected-(J1-Pad16)
- J1 pad 17: (no net) -> unconnected-(J1-Pad17)
- J1 pad 18: (no net) -> unconnected-(J1-Pad18)
- J1 pad 19: (no net) -> unconnected-(J1-Pad19)
- J1 pad 21: (no net) -> unconnected-(J1-Pad21)
- J1 pad 23: (no net) -> unconnected-(J1-Pad23)
- J1 pad 25: (no net) -> unconnected-(J1-Pad25)
- J1 pad 27: (no net) -> unconnected-(J1-Pad27)
- J1 pad 29: (no net) -> unconnected-(J1-Pad29)
- J1 pad 31: (no net) -> unconnected-(J1-Pad31)
- J1 pad 33: (no net) -> unconnected-(J1-Pad33)
- J1 pad 36: (no net) -> unconnected-(J1-Pad36)
- J1 pad 38: (no net) -> unconnected-(J1-Pad38)
- J1 pad 7: (no net) -> unconnected-(J1-Pad7)
- J12 pad 1: (no net) -> unconnected-(J12-Pad1)
- J12 pad 4: (no net) -> unconnected-(J12-Pad4)
- J7 pad 1: (no net) -> unconnected-(J7-Pad1)
- J7 pad 2: (no net) -> unconnected-(J7-Pad2)
- J8 pad 4: (no net) -> unconnected-(J8-Pad4)
- J8 pad 5: (no net) -> unconnected-(J8-Pad5)
- J9 pad 5: (no net) -> unconnected-(J9-Pad5)
Routing:
- net +3V3: track 284.8 -> 281.3 mm
- net /mcu_uart2_rx: track 36.8 -> 35.2 mm
- net /mcu_uart2_tx: track 41.4 -> 39.9 mm
- net /mcu_pb14: track 42.0 -> 40.8 mm
- net /~{mcu_spi1_cs2}: track 65.1 -> 64.4 mm
- net /mcu_adc14: track 49.2 -> 48.6 mm
- net GND: track 5.26 -> 4.67 mm
- net /mcu_pb1: track 44.1 -> 43.6 mm
- net /mcu_pc8: track 60.6 -> 60.1 mm
- net /mcu_pb15: track 41.3 -> 40.8 mm
Other:
- outline, holes or cut-outs redrawn
- net class Default removed
- net class Supply removed
- board text added: "PMI-BoB² V1.3 2023"
- board text added: "~{CS}"
- board text added: "~{SPI1 }CS1"
- board text added: "~{SPI1 }CS2"
- board text added: "~{SPI1_CS1}"
- board text added: "~{SPI1_CS2}"
- board text removed: "PMI-BoB² V1.2 2021"
- board text removed: "~CS"
- board text removed: "~SPI1 ~CS1"
- board text removed: "~SPI1 ~CS2"
- board text removed: "~SPI1_CS1"
- board text removed: "~SPI1_CS2"
